File: controller/controller.kicad_pcb (KiCad board)
At the start: 2 copper layers, 50 x 23 mm, 32 parts, among them J1 ICSP, J2 USB_B_Micro, J3 TRRS_Jack, J4 6P_ZH_connector, J5 6P_ZH_connector, SW1 RESET, U3 ATmega32U4-AU, Y1 16MHz

Commit message: [fix] D-/D+ flip [add] smd jumper for Tx/Rx selection
Parts:
- added JP1: Jumper_right_Tx, MyLib:soldering_jumper_W0.8_P0.2, F.Cu at (95.8, 63.7)
- added JP2: Jumper_right_Rx, MyLib:soldering_jumper_W0.8_P0.2, F.Cu at (94.7, 63.7)
- added JP3: Jumper_left_Rx, MyLib:soldering_jumper_W0.8_P0.2, B.Cu at (95.7, 63.7)
- added JP4: Jumper_left_Tx, MyLib:soldering_jumper_W0.8_P0.2, B.Cu at (96.8, 63.7)
- moved REF** 8.23 mm to (73.0, 53.9)
Connections:
- J3 pad R1: /Rx -> Net-(J3-PadR1)
- J3 pad R2: /Tx -> Net-(J3-PadR2)
- U3 pad 3: /D+ -> /D-
- U3 pad 4: /D- -> /D+
Routing:
- net Net-(J3-PadR2): track 0.00 -> 22.6 mm
- net Net-(J3-PadR1): track 0.00 -> 14.6 mm
- net /Tx: track 31.1 -> 22.6 mm, vias 0 -> 1
- net /Rx: track 25.4 -> 18.8 mm, vias 0 -> 1
- net /D+: track 18.6 -> 20.1 mm
- net /D-: track 23.2 -> 24.6 mm
Other:
- board text added: "Short here for Lefthand"
- board text added: "Short here for Righthand"
- board text added: "Splitify"
- board text added: "rev 3.0"
- board text removed: "For: Lefthand"
- board text removed: "Split HHKB"
- board text removed: "rev 1.0"
